Commit message: add new rules for the gripper

File: urdf/end_effectors/rh_p12_rn_a/rh_p12_rn_a_macro.urdf.xacro (robot description, xacro)
@@ -1,5 +1,5 @@
 <?xml version="1.0"?>
 <robot xmlns:xacro="http://www.ros.org/wiki/xacro">
-  <xacro:macro name="rh_p12_gripper" params="parent prefix:='' use_sim:='false' use_fake_hardware:='false' fake_sensor_commands:='false' ros2_control:='true' *origin">
+  <xacro:macro name="rh_p12_gripper" params="parent prefix:='' port_name:='/dev/ttyUSB0' use_sim:='false' use_fake_hardware:='false' fake_sensor_commands:='false' ros2_control:='true' *origin">
     <!-- Include the definitions -->
     <xacro:include filename="$(find franka_robot_description)/urdf/end_effectors/rh_p12_rn_a/rh_p12_rn_a.xacro" />
@@ -19,4 +19,5 @@
         name="RH_P12_RN_A_System"
         prefix="${prefix}"
+        port_name="${port_name}"
         use_sim="${use_sim}"
         use_fake_hardware="${use_fake_hardware}"

File: urdf/main_assemblies/bimanual_dfki.urdf.xacro (robot description, xacro)
@@ -16,4 +16,5 @@
   <!-- "none", "franka_default", "rh_p12_rn_a" -->
   <xacro:arg name="gripper_type" default="franka_default" />
+  <xacro:arg name="port_name" default="/dev/ttyUSB0" />
   <xacro:arg name="parent" default="world" />
   <xacro:arg name="ros2_control" default="true" />
@@ -71,4 +72,5 @@
         parent="${modified_prefix}$(arg arm_id)_link8"
         prefix="${modified_prefix}"
+        port_name="$(arg port_name)"
         use_fake_hardware="$(arg use_fake_hardware)"
         fake_sensor_commands="$(arg fake_sensor_commands)"
