Commit message: fix: 2s gripper comms timeout, passive grasp_point, ZED wrist mount geometry
- rh_p12_rn_a: error_timeout_ms 500 -> 2000; the long gripper cables drop
  replies in bursts and 500 ms took the left gripper down.
- bimanual_dfki: any gripper_type other than franka_default / rh_p12_rn_a now
  gets a passive grasp_point at the xyz_ee offset, so end_effector_frame
  resolves whatever is fitted. port_name arg renamed to gripper_port.
- Cameras are no longer tied to rh_p12_rn_a: camera_name defaults to 'none'
  and the mount link comes from camera_holder_parent_frame.
- zed_macro: measured wrist-mount geometry; zed_*_base_link renamed to
  zed_*_camera_link.

File: urdf/cameras/zed/zed_descr.urdf.xacro (robot description, xacro)
@@ -18,5 +18,5 @@
   <xacro:arg name="camera_name"   default="zed" />
   <xacro:arg name="camera_model"  default="zed" />
-  <xacro:arg name="base_frame"    default="base_link" />
+  <xacro:arg name="camera_holder_parent_frame" default="base_link" />
   <xacro:arg name="cam_pos_x"     default="0.0" />
   <xacro:arg name="cam_pos_y"     default="0.0" />
@@ -27,5 +27,5 @@
   <xacro:arg name="gnss_frame"    default="" />
   <xacro:include filename="$(find franka_robot_description)/urdf/cameras/zed/zed_macro.urdf.xacro" />
-  <xacro:zed_camera name="$(arg camera_name)" model="$(arg camera_model)" parent="$(arg base_frame)">
+  <xacro:zed_camera name="$(arg camera_name)" model="$(arg camera_model)" parent="$(arg camera_holder_parent_frame)">
     <origin
       xyz="$(arg cam_pos_x) $(arg cam_pos_y) $(arg cam_pos_z)"
@@ -33,4 +33,4 @@
     />
   </xacro:zed_camera>
-  <link name="$(arg base_frame)" />
+  <link name="$(arg camera_holder_parent_frame)" />
 </robot>

File: urdf/cameras/zed/zed_macro.urdf.xacro (robot description, xacro)
@@ -22,5 +22,5 @@
       - name: the camera's name.  should match the parameter sent to the launch file for this camera
       - model: the tye of camera, one of zed, zedm, zed2, zed2i
-      - parent: the parent link of the camera.  must be defined in the URDF file that uses this macro
+      - parent: the parent link of the camera holder.  must be defined in the URDF file that uses this macro
       - origin: the xyz/rpy offset from the parent link
   -->
@@ -95,12 +95,12 @@
       <parent link="${parent}"/>
       <child link="${name}_camera_holder"/>
-      <origin xyz="0 0 0.00255" rpy="${M_PI} 0 -${M_PI/4}" />
+      <origin xyz="0 0 0.00255" rpy="${M_PI} 0 ${3*M_PI/4}" />
       <xacro:insert_block name="origin" />
     </joint>
-    <link name="${name}_base_link" />
-    <joint name="${name}_base_joint" type="fixed">
+    <link name="${name}_camera_link" />
+    <joint name="${name}_camera_link_joint" type="fixed">
       <parent link="${name}_camera_holder"/>
-      <child link="${name}_base_link"/>
-      <origin xyz="-0.093473 0 -0.015021" rpy="0 0 0" />
+      <child link="${name}_camera_link"/>
+      <origin xyz="-0.085473 0 -0.016021" rpy="${M_PI} 0.873 0" />
     </joint>
     <!-- Camera Center -->
@@ -114,4 +114,5 @@
       </visual>
       <collision>
+        <origin xyz="${screw_offset_x} 0 ${screw_offset_z}" rpy="0 0 0"/>
         <geometry>
           <mesh filename="package://franka_robot_description/meshes/cameras/zed/${model}.stl" />
@@ -125,7 +126,7 @@
     </link>
     <joint name="${name}_camera_center_joint" type="fixed">
-      <parent link="${name}_base_link"/>
+      <parent link="${name}_camera_link"/>
       <child link="${name}_camera_center"/>
-      <origin xyz="0 0 -${height/2}" rpy="0 0.85 0" />
+      <origin xyz="0 0 ${height/2}" rpy="0 ${bottom_slope} 0" />
     </joint>
     <!-- Left Camera -->

File: urdf/end_effectors/rh_p12_rn_a/rh_p12_rn_a.ros2_control.xacro (robot description, xacro)
@@ -19,5 +19,6 @@
             <param name="port_name">${port_name}</param>
             <param name="baud_rate">2000000</param>
-            <param name="error_timeout_ms">500</param>
+            <!-- 2 s: the long gripper cables drop replies in bursts; 500 ms took the left gripper down. -->
+            <param name="error_timeout_ms">2000</param>
             <param name="dynamixel_model_folder">/param/dxl_model</param>
             <param name="number_of_joints">1</param>

File: urdf/main_assemblies/bimanual_dfki.urdf.xacro (robot description, xacro)
@@ -14,14 +14,15 @@
   <xacro:arg name="xyz_ee" default="0 0 0" />
   <xacro:arg name="rpy_ee" default="0 0 0" />
-  <!-- "none", "franka_default", "rh_p12_rn_a" -->
+  <!-- "franka_default", "rh_p12_rn_a", or anything else for a passive end-effector -->
   <xacro:arg name="gripper_type" default="franka_default" />
-  <xacro:arg name="port_name" default="/dev/ttyUSB0" />
+  <xacro:arg name="gripper_port" default="/dev/ttyUSB0" />
   <xacro:arg name="parent" default="world" />
   <xacro:arg name="ros2_control" default="true" />
   <xacro:arg name="gripper_ros2_control" default="true" />
   <xacro:arg name="gazebo" default="false" />
-  <xacro:arg name="camera_name" default="zed" />
+  <!-- Camera mounted on this arm; 'none' means this arm carries no camera. -->
+  <xacro:arg name="camera_name" default="none" />
   <xacro:arg name="camera_model" default="zedxm" />
-  <xacro:arg name="base_frame"    default="base_link" />
+  <xacro:arg name="camera_holder_parent_frame" default="fr3_link8" />
   <xacro:arg name="cam_pos_x"     default="0.0" />
   <xacro:arg name="cam_pos_y"     default="0.0" />
@@ -30,5 +31,4 @@
   <xacro:arg name="cam_pitch"     default="0.0" />
   <xacro:arg name="cam_yaw"       default="0.0" />
-  <xacro:arg name="gnss_frame"    default="" />
   <!-- ============================================== -->
   <!-- Property Processing                            -->
@@ -72,8 +72,8 @@
         parent="${modified_prefix}$(arg arm_id)_link8"
         prefix="${modified_prefix}"
-        port_name="$(arg port_name)"
         use_fake_hardware="$(arg use_fake_hardware)"
         fake_sensor_commands="$(arg fake_sensor_commands)"
         ros2_control="$(arg gripper_ros2_control)"
+        port_name="$(arg gripper_port)"
         use_sim="$(arg use_sim)">
         <origin xyz="$(arg xyz_ee)" rpy="$(arg rpy_ee)"/>
@@ -83,7 +83,7 @@
   <!-- Zed Camera Attachments                    -->
   <!-- ============================================== -->
-  <xacro:if value="${'$(arg camera_name)' == 'zed' and '$(arg gripper_type)' == 'rh_p12_rn_a'}">
+  <xacro:if value="${'$(arg camera_name)' != 'none'}">
     <xacro:include filename="$(find franka_robot_description)/urdf/cameras/zed/zed_macro.urdf.xacro" />
-    <xacro:zed_camera name="$(arg camera_name)" model="$(arg camera_model)" parent="${modified_prefix}$(arg arm_id)_link8">
+    <xacro:zed_camera name="$(arg camera_name)" model="$(arg camera_model)" parent="${modified_prefix}$(arg camera_holder_parent_frame)">
       <origin
         xyz="$(arg cam_pos_x) $(arg cam_pos_y) $(arg cam_pos_z)"
@@ -111,3 +111,13 @@
     </joint>
   </xacro:if>
+  <!-- Anything else is a passive end-effector: grasp_point sits at the xyz_ee/rpy_ee
+       offset from the flange, so end_effector_frame resolves whatever is fitted. -->
+  <xacro:if value="${'$(arg gripper_type)' not in ['franka_default', 'rh_p12_rn_a']}">
+    <link name="${modified_prefix}grasp_point" />
+    <joint name="${modified_prefix}grasp_point_joint" type="fixed">
+      <parent link="${modified_prefix}$(arg arm_id)_link8" />
+      <child link="${modified_prefix}grasp_point" />
+      <origin xyz="$(arg xyz_ee)" rpy="$(arg rpy_ee)" />
+    </joint>
+  </xacro:if>
 </robot>
