Commit message: Update camera config and bimanual config

File: urdf/cameras/zed/zed_macro.urdf.xacro (robot description, xacro)
@@ -23,7 +23,11 @@
       - model: the tye of camera, one of zed, zedm, zed2, zed2i
       - parent: the parent link of the camera.  must be defined in the URDF file that uses this macro
-      - origin: the xyz/rpy offset from the parent link
+      - origin: the xyz/rpy offset from the parent link (a correction applied before the holder)
+      - holder_yaw: yaw of the holder about the flange axis (both wrist mounts: -pi/4)
+      - image_flip: the published images are turned by 180 deg about the optical axis relative to
+        the mounted camera (measured on the wrist ZED X Minis: the table only comes out level
+        with it), so the optical frames are rolled by pi
   -->
-  <xacro:macro name="zed_camera" params="name=zed model=zed parent *origin">
+  <xacro:macro name="zed_camera" params="name=zed model=zed parent holder_yaw:=${-M_PI/4} image_flip:=false *origin">
     <xacro:if value="${model == 'zed'}">
       <xacro:property name="baseline" value="0.12" />
@@ -92,9 +96,16 @@
       </collision>
     </link>
+    <!-- The origin block: a correction of the whole camera in the parent frame (zero for the
+         nominal mount; written by scripts/python/board_calibration.py for the wrist cameras) -->
+    <link name="${name}_camera_mount" />
+    <joint name="${name}_mount_joint" type="fixed">
+      <parent link="${parent}"/>
+      <child link="${name}_camera_mount"/>
+      <xacro:insert_block name="origin" />
+    </joint>
     <joint name="${name}_holder_joint" type="fixed">
-      <parent link="${parent}"/>
+      <parent link="${name}_camera_mount"/>
       <child link="${name}_camera_holder"/>
-      <origin xyz="0 0 0.00255" rpy="${M_PI} 0 -${M_PI/4}" />
-      <xacro:insert_block name="origin" />
+      <origin xyz="0 0 0.00255" rpy="${M_PI} 0 ${holder_yaw}" />
     </joint>
     <link name="${name}_base_link" />
@@ -138,5 +149,5 @@
     <link name="${name}_left_camera_optical_frame"/>
     <joint name="${name}_left_camera_optical_joint" type="fixed">
-      <origin xyz="0 0 0" rpy="-${M_PI/2} 0.0 -${M_PI/2}"/>
+      <origin xyz="0 0 0" rpy="${M_PI/2 if image_flip else -M_PI/2} 0.0 ${M_PI/2 if image_flip else -M_PI/2}"/>
       <parent link="${name}_left_camera_frame"/>
       <child link="${name}_left_camera_optical_frame"/>
@@ -151,5 +162,5 @@
     <link name="${name}_right_camera_optical_frame"/>
     <joint name="${name}_right_camera_optical_joint" type="fixed">
-      <origin xyz="0 0 0" rpy="-${M_PI/2} 0.0 -${M_PI/2}"/>
+      <origin xyz="0 0 0" rpy="${M_PI/2 if image_flip else -M_PI/2} 0.0 ${M_PI/2 if image_flip else -M_PI/2}"/>
       <parent link="${name}_right_camera_frame"/>
       <child link="${name}_right_camera_optical_frame"/>

File: urdf/main_assemblies/bimanual_dfki.urdf.xacro (robot description, xacro)
@@ -30,4 +30,7 @@
   <xacro:arg name="cam_pitch"     default="0.0" />
   <xacro:arg name="cam_yaw"       default="0.0" />
+  <!-- Wrist ZED mount (zed_macro.urdf.xacro): holder yaw on the flange, images turned by pi -->
+  <xacro:arg name="cam_holder_yaw" default="-0.785398163" />
+  <xacro:arg name="cam_image_flip" default="true" />
   <xacro:arg name="gnss_frame"    default="" />
   <!-- ============================================== -->
@@ -85,5 +88,8 @@
   <xacro:if value="${'$(arg camera_name)' == 'zed' and '$(arg gripper_type)' == 'rh_p12_rn_a'}">
     <xacro:include filename="$(find franka_robot_description)/urdf/cameras/zed/zed_macro.urdf.xacro" />
-    <xacro:zed_camera name="$(arg camera_name)" model="$(arg camera_model)" parent="${modified_prefix}$(arg arm_id)_link8">
+    <!-- Prefixed like the arm: both wrist cameras share camera_name, and unprefixed frames
+         (zed_left_camera_optical_frame, ...) collide on /tf_static between the two robots. -->
+    <xacro:zed_camera name="${modified_prefix}$(arg camera_name)" model="$(arg camera_model)" parent="${modified_prefix}$(arg arm_id)_link8"
+                      holder_yaw="$(arg cam_holder_yaw)" image_flip="$(arg cam_image_flip)">
       <origin
         xyz="$(arg cam_pos_x) $(arg cam_pos_y) $(arg cam_pos_z)"

Commit message: Add updated camera holder

File: urdf/cameras/zed/zed_macro.urdf.xacro (robot description, xacro)
@@ -25,9 +25,13 @@
       - origin: the xyz/rpy offset from the parent link (a correction applied before the holder)
       - holder_yaw: yaw of the holder about the flange axis (both wrist mounts: -pi/4)
+      - holder: the wrist holder, "default" (zed_holder.stl: camera on a ~40 deg seat 93 mm off the
+        flange axis) or "short" (zed_holder_short.stl, "close": camera bottom on a vertical wall
+        49 mm off the axis, looking along the gripper). The short pose is nominal from the CAD
+        (wall face, screw height); the board calibration corrects it through the origin block.
       - image_flip: the published images are turned by 180 deg about the optical axis relative to
         the mounted camera (measured on the wrist ZED X Minis: the table only comes out level
         with it), so the optical frames are rolled by pi
   -->
-  <xacro:macro name="zed_camera" params="name=zed model=zed parent holder_yaw:=${-M_PI/4} image_flip:=false *origin">
+  <xacro:macro name="zed_camera" params="name=zed model=zed parent holder_yaw:=${-M_PI/4} holder:=default image_flip:=false *origin">
     <xacro:if value="${model == 'zed'}">
       <xacro:property name="baseline" value="0.12" />
@@ -78,4 +82,24 @@
       <xacro:property name="optical_offset_x" value="-0.01" />
     </xacro:if>
+    <!-- Holder geometry: mesh, camera screw point (base_link) and camera centre relative to it -->
+    <xacro:if value="${holder == 'default'}">
+      <xacro:property name="holder_mesh" value="zed_holder.stl" />
+      <xacro:property name="holder_scale" value="1 1 1" />
+      <xacro:property name="base_xyz" value="-0.093473 0 -0.015021" />
+      <xacro:property name="center_xyz" value="0 0 -${height/2}" />
+      <xacro:property name="center_pitch" value="0.85" />
+    </xacro:if>
+    <xacro:if value="${holder == 'short'}">
+      <!-- Wall face x = -49.37 mm - 0.0462 z (2.6 deg), centre screw at z = -14.2 mm; the camera
+           centre half a camera height out of the wall, its up axis into the wall. -->
+      <xacro:property name="holder_mesh" value="zed_holder_short.stl" />
+      <xacro:property name="holder_scale" value="0.001 0.001 0.001" />
+      <xacro:property name="base_xyz" value="-0.048714 0 -0.0142" />
+      <xacro:property name="center_xyz" value="${-0.99893 * height/2} 0 ${-0.04615 * height/2}" />
+      <xacro:property name="center_pitch" value="1.52463" />
+    </xacro:if>
+    <xacro:unless value="${holder in ('default', 'short')}">
+      <xacro:property name="holder_unknown" lazy_eval="false" value="${xacro.fatal('zed_camera: unknown holder ' + str(holder) + ' (default | short)')}" />
+    </xacro:unless>
     <!-- Camera mounting point (the threaded screw hole in the bottom) -->
     <link name="${name}_camera_holder">
@@ -83,5 +107,5 @@
         <origin xyz="0 0 0" rpy="0 0 0"/>
         <geometry>
-          <mesh filename="package://franka_robot_description/meshes/cameras/zed/zed_holder.stl" />
+          <mesh filename="package://franka_robot_description/meshes/cameras/zed/${holder_mesh}" scale="${holder_scale}" />
         </geometry>
         <material name="red">
@@ -92,5 +116,5 @@
         <origin xyz="0 0 0" rpy="0 0 0"/>
         <geometry>
-          <mesh filename="package://franka_robot_description/meshes/cameras/zed/zed_holder.stl" />
+          <mesh filename="package://franka_robot_description/meshes/cameras/zed/${holder_mesh}" scale="${holder_scale}" />
         </geometry>
       </collision>
@@ -113,5 +137,5 @@
       <parent link="${name}_camera_holder"/>
       <child link="${name}_base_link"/>
-      <origin xyz="-0.093473 0 -0.015021" rpy="0 0 0" />
+      <origin xyz="${base_xyz}" rpy="0 0 0" />
     </joint>
     <!-- Camera Center -->
@@ -138,5 +162,5 @@
       <parent link="${name}_base_link"/>
       <child link="${name}_camera_center"/>
-      <origin xyz="0 0 -${height/2}" rpy="0 0.85 0" />
+      <origin xyz="${center_xyz}" rpy="0 ${center_pitch} 0" />
     </joint>
     <!-- Left Camera -->

File: urdf/main_assemblies/bimanual_dfki.urdf.xacro (robot description, xacro)
@@ -33,4 +33,6 @@
   <xacro:arg name="cam_holder_yaw" default="-0.785398163" />
   <xacro:arg name="cam_image_flip" default="true" />
+  <!-- Wrist holder: default (zed_holder.stl) | short (zed_holder_short.stl, camera closer to the flange) -->
+  <xacro:arg name="camera_holder" default="default" />
   <xacro:arg name="gnss_frame"    default="" />
   <!-- ============================================== -->
@@ -91,5 +93,5 @@
          (zed_left_camera_optical_frame, ...) collide on /tf_static between the two robots. -->
     <xacro:zed_camera name="${modified_prefix}$(arg camera_name)" model="$(arg camera_model)" parent="${modified_prefix}$(arg arm_id)_link8"
-                      holder_yaw="$(arg cam_holder_yaw)" image_flip="$(arg cam_image_flip)">
+                      holder_yaw="$(arg cam_holder_yaw)" holder="$(arg camera_holder)" image_flip="$(arg cam_image_flip)">
       <origin
         xyz="$(arg cam_pos_x) $(arg cam_pos_y) $(arg cam_pos_z)"
